File: type-c_plug_lipo.kicad_pcb (KiCad board)
At the start: 2 copper layers, 27.1 x 20 mm, 20 parts, among them J1 Conn_Battery, J2 USB_C_Plug_USB2.0, J4 Conn_Pwr, U1 MCP73831

Commit message: Rev 2
Parts:
- U1: value MCP73831 -> ME4055-N; footprint Package_TO_SOT_SMD:SOT-23-5 -> Package_TO_SOT_SMD:SOT-23-6
Connections:
- D2 pad 1: GND -> Net-(D2-Pad1)
- D2 pad 2: Net-(D2-Pad2) -> VBUS
- J2 pad B5: Net-(J2-PadB5) -> unconnected-(J2-PadB5)
- R4 pad 1: Net-(R3-Pad1) -> Net-(R4-Pad1)
- R4 pad 2: Net-(D2-Pad2) -> Net-(D2-Pad1)
- U1 pad 5: Net-(R2-Pad2) -> Net-(R4-Pad1)
Routing:
- net Net-(R4-Pad1): track 0.00 -> 8.01 mm, vias 0 -> 2
- net Net-(D2-Pad1): track 0.00 -> 5.76 mm
- net Net-(D2-Pad2): track 4.59 -> 0.00 mm
- net Net-(R3-Pad1): track 3.49 -> 2.09 mm
- net VBUS: track 29.8 -> 31.2 mm
Other:
- board text added: "3.7V LiPo Charger Charge: 4.2V @ 600mA by arturo182 Dec 2022"
- board text removed: "3.7V LiPo Charger Charge: 4.2V @ 500mA by arturo182 Oct 2020"
